File: XO2-DIP20/XO2-DIP20.kicad_pcb (KiCad board)
At the start: 2 copper layers, 10.2 x 25.4 mm, 6 parts, among them J2 Conn_02x03_Odd_Even, U1 MachXO2-1200

Commit message: Finish PCB design
Parts:
- added R1: 4k7, Resistor_SMD:R_0603_1608Metric_Pad0.98x0.95mm_HandSolder, F.Cu at (127.0, 68.0)
- moved C1 0.34 mm to (127.0, 79.3)
- moved C2 0.22 mm to (127.0, 77.5)
Connections:
- JL1 pad 4: /PIN9 -> /PIN8
- JL1 pad 5: /PIN8 -> /PIN9
- JR1 pad 6: /PIN26 -> /PIN25
- JR1 pad 7: /PIN27 -> /PIN26
- JR1 pad 8: /PIN25 -> /PIN27
Routing:
- net /PIN25: track 7.79 -> 1.17 mm
- net /PIN8: track 1.17 -> 5.38 mm
- net /PIN27: track 3.26 -> 6.89 mm
- net /PIN9: track 5.69 -> 2.47 mm, vias 0 -> 1
- net /PIN26: track 1.38 -> 3.65 mm, vias 0 -> 1
- net /TCK: track 4.84 -> 6.97 mm
- net /TDO: track 3.70 -> 4.56 mm
- net GND: track 5.37 -> 6.15 mm, vias 2 -> 3
Other:
- board text added: "10"
- board text added: "11"
- board text added: "12"
- board text added: "13"
- board text added: "14"
- board text added: "16"
- board text added: "17"
- board text added: "20"
- board text added: "21"
- board text added: "23"
- board text added: "25"
- board text added: "26"
- board text added: "27"
- board text added: "28"
- board text added: "4"
- board text added: "5"
- board text added: "8"
- board text added: "9"
- board text added: "G"
- board text added: "GND VCC TDI TMS TDO TCK"
- board text added: "MachXO2-DIP20 Rev1 ©2023 c0pperdragon"
- board text added: "V"
