File: XO2-DIP20/XO2-DIP20.kicad_sch (KiCad schematic)
At the start: 6 parts, among them J2 Conn_02x03_Odd_Even, U1 MachXO2-1200

Commit message: Finish PCB design
Parts:
- added R1: 4k7, Resistor_SMD:R_0603_1608Metric_Pad0.98x0.95mm_HandSolder, symbol Device:R_Small
Connections:
- net GND: now also R1.2
- net PIN25: now also JR1.6 (Pin_6); no longer JR1.8 (Pin_8)
- net PIN26: now also JR1.7 (Pin_7); no longer JR1.6 (Pin_6)
- net PIN27: now also JR1.8 (Pin_8); no longer JR1.7 (Pin_7)
- net PIN8: now also JL1.4 (Pin_4); no longer JL1.5 (Pin_5)
- net PIN9: now also JL1.5 (Pin_5); no longer JL1.4 (Pin_4)
- net TCK: now also R1.1
Changed lines of the file:
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@@
 (kicad_sch (version 20211123) (generator eeschema)
   (paper "A4")
+  (junction (at 114.3 93.98) (diameter 0) (color 0 0 0 0)
+  )
   (junction (at 44.45 149.86) (diameter 0) (color 0 0 0 0)
   )
@@
     (stroke (width 0) (type default) (color 0 0 0 0))
   )
+  (wire (pts (xy 114.3 93.98) (xy 114.3 116.84))
+    (stroke (width 0) (type default) (color 0 0 0 0))
+  )
   (wire (pts (xy 121.92 88.9) (xy 129.54 88.9))
     (stroke (width 0) (type default) (color 0 0 0 0))
   )
+  (wire (pts (xy 114.3 93.98) (xy 129.54 93.98))
+    (stroke (width 0) (type default) (color 0 0 0 0))
+  )
   (wire (pts (xy 40.64 77.47) (xy 41.91 77.47))
     (stroke (width 0) (type default) (color 0 0 0 0))
@@
     (stroke (width 0) (type default) (color 0 0 0 0))
   )
+  (wire (pts (xy 114.3 121.92) (xy 114.3 124.46))
+    (stroke (width 0) (type default) (color 0 0 0 0))
+  )
   (wire (pts (xy 44.45 149.86) (xy 55.88 149.86))
     (stroke (width 0) (type default) (color 0 0 0 0))
@@
     (stroke (width 0) (type default) (color 0 0 0 0))
   )
-  (wire (pts (xy 109.22 93.98) (xy 129.54 93.98))
+  (wire (pts (xy 109.22 93.98) (xy 114.3 93.98))
     (stroke (width 0) (type default) (color 0 0 0 0))
   )
@@
     (effects (font (size 1.27 1.27)) (justify right bottom))
   )
-  (label "PIN8" (at 35.56 87.63 0)
+  (label "PIN8" (at 35.56 85.09 0)
     (effects (font (size 1.27 1.27)) (justify left bottom))
   )
@@
     (effects (font (size 1.27 1.27)) (justify left bottom))
   )
-  (label "PIN25" (at 82.55 82.55 180)
+  (label "PIN25" (at 82.55 87.63 180)
     (effects (font (size 1.27 1.27)) (justify right bottom))
   )
@@
     (effects (font (size 1.27 1.27)) (justify left bottom))
   )
-  (label "PIN26" (at 82.55 87.63 180)
+  (label "PIN26" (at 82.55 85.09 180)
     (effects (font (size 1.27 1.27)) (justify right bottom))
   )
@@
     (effects (font (size 1.27 1.27)) (justify left bottom))
   )
-  (label "PIN9" (at 35.56 85.09 0)
+  (label "PIN9" (at 35.56 87.63 0)
     (effects (font (size 1.27 1.27)) (justify left bottom))
   )
@@
     (effects (font (size 1.27 1.27)) (justify left bottom))
   )
-  (label "PIN27" (at 82.55 85.09 180)
+  (label "PIN27" (at 82.55 82.55 180)
     (effects (font (size 1.27 1.27)) (justify right bottom))
   )
@@
     (pin "1")
   )
+  (symbol (lib_id "Device:R_Small") (at 114.3 119.38 0) (unit 1)
+    (in_bom yes) (on_board yes) (fields_autoplaced)
+    (property "Reference" "R1" (id 0) (at 116.84 118.1099 0)
+      (effects (font (size 1.27 1.27)) (justify left))
+    )
+    (property "Value" "4k7" (id 1) (at 116.84 120.6499 0)
+      (effects (font (size 1.27 1.27)) (justify left))
+    )
+    (property "Footprint" "Resistor_SMD:R_0603_1608Metric_Pad0.98x0.95mm_HandSolder" (id 2) (at 114.3 119.38 0)
+      (effects (font (size 1.27 1.27)) hide)
+    )
+    (property "Datasheet" "~" (id 3) (at 114.3 119.38 0)
+      (effects (font (size 1.27 1.27)) hide)
+    )
+    (pin "1")
+    (pin "2")
+  )
   (symbol (lib_id "Device:C_Small") (at 55.88 154.94 0) (unit 1)
     (in_bom yes) (on_board yes) (fields_autoplaced)
@@
     )
     (property "Datasheet" "" (id 3) (at 44.45 147.32 0)
+      (effects (font (size 1.27 1.27)) hide)
+    )
+    (pin "1")
+  )
+  (symbol (lib_id "power:GND") (at 114.3 124.46 0) (unit 1)
+    (in_bom yes) (on_board yes) (fields_autoplaced)
+    (property "Reference" "#PWR0116" (id 0) (at 114.3 130.81 0)
+      (effects (font (size 1.27 1.27)) hide)
+    )
+    (property "Value" "GND" (id 1) (at 114.3 129.54 0))
+    (property "Footprint" "" (id 2) (at 114.3 124.46 0)
+      (effects (font (size 1.27 1.27)) hide)
+    )
+    (property "Datasheet" "" (id 3) (at 114.3 124.46 0)
       (effects (font (size 1.27 1.27)) hide)
     )
@@
       (reference "#PWR0115") (unit 1) (value "VCC") (footprint "")
     )
+    (path "/ce164a52-026e-467b-8ade-7b086ff2cddc"
+      (reference "#PWR0116") (unit 1) (value "GND") (footprint "")
+    )
     (path "/ae75d6d4-068a-4f90-9cbc-b0a5614968d0"
       (reference "#PWR0117") (unit 1) (value "VCC") (footprint "")
@@
       (reference "JR1") (unit 1) (value "Conn_01x10") (footprint "Connector_PinHeader_2.54mm:PinHeader_1x10_P2.54mm_Vertical")
     )
+    (path "/a0f6ba91-4251-44e7-91f1-dd32d453baa6"
+      (reference "R1") (unit 1) (value "4k7") (footprint "Resistor_SMD:R_0603_1608Metric_Pad0.98x0.95mm_HandSolder")
+    )
     (path "/2b2b0393-ee56-4368-bad7-0995a69d5218"
